Commit message: updated camera position

File: clearpath_jackal_description/robot.srdf.xacro (robot description, xacro)
@@ -2,13 +2,5 @@
 <robot xmlns:xacro="http://www.ros.org/wiki/xacro" name="j100-0897">
   <!-- Arms -->
-  <!-- arm_0 -->
-  <xacro:include filename="$(find clearpath_manipulators_description)/srdf/arm/kinova_gen3_lite.srdf.xacro"/>
-  <xacro:kinova_gen3_lite_group_state name="arm_0" group_state="custom" joint_positions="${[0.0000, 0.0000, 0.0000, 0.0000, 0.0000, 0.0000]}"/>
-  <xacro:kinova_gen3_lite name="arm_0"/>
   <!-- Grippers -->
-  <!-- arm_0_gripper -->
-  <xacro:include filename="$(find clearpath_manipulators_description)/srdf/gripper/kinova_2f_lite.srdf.xacro"/>
-  <xacro:kinova_2f_lite_group_state name="arm_0_gripper" group_state="custom" joint_positions="${[0.0000]}"/>
-  <xacro:kinova_2f_lite name="arm_0_gripper"/>
   <!-- Lifts -->
 </robot>

File: clearpath_jackal_description/robot.urdf.xacro (robot description, xacro)
@@ -44,18 +44,13 @@
   <!-- camera_0 -->
   <xacro:include filename="$(find clearpath_sensors_description)/urdf/intel_realsense.urdf.xacro"/>
-  <xacro:intel_realsense name="camera_0" parent_link="base_link" update_rate="30" image_height="480" image_width="640" model="d435">
+  <xacro:intel_realsense name="camera_0" parent_link="front_fender_mount" update_rate="30" image_height="480" image_width="640" model="d435">
+    <origin xyz="0.01 0.0 -0.05" rpy="3.1415 0.0 0.0"/>
+  </xacro:intel_realsense>
+  <!-- imu_1 -->
+  <xacro:include filename="$(find clearpath_sensors_description)/urdf/redshift_um7.urdf.xacro"/>
+  <xacro:redshift_um7 name="imu_1" parent_link="base_link" update_rate="20">
     <origin xyz="0.0 0.0 0.0" rpy="0.0 0.0 0.0"/>
-  </xacro:intel_realsense>
+  </xacro:redshift_um7>
   <!-- Manipulators -->
-  <!-- arm_0 -->
-  <xacro:include filename="$(find clearpath_manipulators_description)/urdf/arm/kinova_gen3_lite.urdf.xacro"/>
-  <xacro:kinova_gen3_lite name="arm_0" parent_link="default_mount" port="10000" robot_ip="192.168.131.40" use_internal_bus_gripper_comm="True" gripper_joint_name="arm_0_gripper_right_finger_bottom_joint">
-    <origin xyz="0.0 0.0 0.0" rpy="0.0 0.0 0.0"/>
-  </xacro:kinova_gen3_lite>
-  <!-- arm_0_gripper -->
-  <xacro:include filename="$(find clearpath_manipulators_description)/urdf/gripper/kinova_2f_lite.urdf.xacro"/>
-  <xacro:kinova_2f_lite name="arm_0_gripper" parent_link="arm_0_end_effector_link">
-    <origin xyz="0.0 0.0 0.0" rpy="0.0 0.0 0.0"/>
-  </xacro:kinova_2f_lite>
   <!-- Extras -->
 </robot>

Commit message: Updated jackal configuration. Mostly working on hardware.

File: clearpath_jackal_description/robot.srdf.xacro (robot description, xacro)
@@ -2,5 +2,13 @@
 <robot xmlns:xacro="http://www.ros.org/wiki/xacro" name="j100-0897">
   <!-- Arms -->
+  <!-- arm_0 -->
+  <xacro:include filename="$(find clearpath_manipulators_description)/srdf/arm/kinova_gen3_lite.srdf.xacro"/>
+  <xacro:kinova_gen3_lite_group_state name="arm_0" group_state="custom" joint_positions="${[0.0000, 0.0000, 0.0000, 0.0000, 0.0000, 0.0000]}"/>
+  <xacro:kinova_gen3_lite name="arm_0"/>
   <!-- Grippers -->
+  <!-- arm_0_gripper -->
+  <xacro:include filename="$(find clearpath_manipulators_description)/srdf/gripper/kinova_2f_lite.srdf.xacro"/>
+  <xacro:kinova_2f_lite_group_state name="arm_0_gripper" group_state="custom" joint_positions="${[0.0000]}"/>
+  <xacro:kinova_2f_lite name="arm_0_gripper"/>
   <!-- Lifts -->
 </robot>

File: clearpath_jackal_description/robot.urdf.xacro (robot description, xacro)
@@ -53,4 +53,14 @@
   </xacro:redshift_um7>
   <!-- Manipulators -->
+  <!-- arm_0 -->
+  <xacro:include filename="$(find clearpath_manipulators_description)/urdf/arm/kinova_gen3_lite.urdf.xacro"/>
+  <xacro:kinova_gen3_lite name="arm_0" parent_link="default_mount" port="10000" robot_ip="192.168.1.10" use_internal_bus_gripper_comm="True" gripper_joint_name="arm_0_gripper_right_finger_bottom_joint">
+    <origin xyz="0.0 0.0 0.0" rpy="0.0 0.0 0.0"/>
+  </xacro:kinova_gen3_lite>
+  <!-- arm_0_gripper -->
+  <xacro:include filename="$(find clearpath_manipulators_description)/urdf/gripper/kinova_2f_lite.urdf.xacro"/>
+  <xacro:kinova_2f_lite name="arm_0_gripper" parent_link="arm_0_end_effector_link">
+    <origin xyz="0.0 0.0 0.0" rpy="0.0 0.0 0.0"/>
+  </xacro:kinova_2f_lite>
   <!-- Extras -->
 </robot>
